Commit message: Changement fonction resetJointState

File: resources/urdf/pps.urdf (robot description, URDF)
Before this commit: robot test_robot, 5 links, 4 joints
Links:
- link A1: mass 0.5 -> 180
- link A2: mass 0.5 -> 299
- link A3: mass 0.5 -> 193.2
- link base: mass 0.0 -> 292.0
Joints:
- joint joint2: origin xyz=35 0 27 rpy=0 0 0 -> xyz=36 0 27 rpy=0 0 0

Commit message: Obtenir des paramètres qui ont du sens (torques, forces,..)

File: resources/urdf/pps.urdf (robot description, URDF)
Before this commit: robot test_robot, 5 links, 4 joints
Links:
- link A1: geometry collision mesh filename=pps_leoni/bras1.obj scale=0.01 0.01 0.01; visual mesh filename=pps_leoni/bras1.obj scale=0.01 0.01 0.01
- link A2: geometry collision mesh filename=pps_leoni/interbras.obj scale=0.01 0.01 0.01; visual mesh filename=pps_leoni/interbras.obj scale=0.01 0.01 0.01
- link A3: geometry collision mesh filename=pps_leoni/BrasExtensionbras2.obj scale=0.01 0.01 0.01; visual mesh filename=pps_leoni/BrasExtensionbras2.obj scale=0.01 0.01 0.01
- link base: geometry collision mesh filename=pps_leoni/pied.obj scale=0.01 0.01 0.01; visual mesh filename=pps_leoni/pied.obj scale=0.01 0.01 0.01
Joints:
- joint base: origin xyz=0.000000 -195.000000 -110.300003 rpy=0 0 0 -> xyz=0.000000 -1.95 -1.10300003 rpy=0 0 0
- joint joint1: origin xyz=-120 0 36 rpy=0 0 0 -> xyz=-1.2 0 0.36 rpy=0 0 0
- joint joint2: origin xyz=36 0 27 rpy=0 0 0 -> xyz=0.36 0 0.27 rpy=0 0 0

File: resources/urdf/urdf_Obstacle.urdf (robot description, URDF)
Before this commit: robot new Obstacle, 2 links, 1 joints
Links:
- link Obstacle: geometry collision box size=0.20 0.20 2; visual box size=0.20 0.20 2.00
Joints:
- joint joint_iso_to_obstacle: origin xyz=100.0 -300.0 10.0 rpy=0 0 0 -> xyz=1 -3 0.10 rpy=0 0 0

Commit message: Modèle 6Dofs avec affichage joint/inertial frames + TCP et closest points

File: resources/urdf/pps.urdf (robot description, URDF)
Before this commit: robot test_robot, 5 links, 4 joints
Links:
- added link A4, mass 41.0; collision mesh filename=pps_leoni/bras3.obj scale=0.01 0.01 0.01; visual mesh filename=pps_leoni/bras3.obj scale=0.01 0.01 0.01
- added link A5, mass 41.6; collision mesh filename=pps_leoni/bras_rot_2.obj scale=0.01 0.01 0.01; visual mesh filename=pps_leoni/bras_rot_2.obj scale=0.01 0.01 0.01
- added link A6, mass 44.0; collision mesh filename=pps_leoni/coupler.obj scale=0.01 0.01 0.01; visual mesh filename=pps_leoni/coupler.obj scale=0.01 0.01 0.01
- added link couch, mass 70.0; collision mesh filename=pps_leoni/couch.obj scale=0.001 0.001 0.001; visual mesh filename=pps_leoni/couch.obj scale=0.001 0.001 0.001
Joints:
- added joint joint3: type continuous, parent A3, child A4, origin xyz=0.980 0 0 rpy=0 0 0, axis -1 0 0
- added joint joint4: type continuous, parent A4, child A5, origin xyz=0.220 0 0 rpy=0 0 0, axis 0 -1 0
- added joint joint5: type continuous, parent A5, child A6, origin xyz=0 0 0.3395 rpy=0 0 0, axis 0 0 1
- added joint joint6: type fixed, parent A6, child couch, origin xyz=-0.36 0 -0.9695 rpy=0 0 0
- joint joint1: origin xyz=-1.2 0 0.36 rpy=0 0 0 -> xyz=-1.2 0 0.4365 rpy=0 0 0
- joint joint2: origin xyz=0.36 0 0.27 rpy=0 0 0 -> xyz=0.36 0 0.1935 rpy=0 0 0

Commit message: Modèle 6Dofs avec joint/inertial frames + TCP correction

File: resources/urdf/pps.urdf (robot description, URDF)
Before this commit: robot test_robot, 9 links, 8 joints
Joints:
- joint base: origin xyz=0.000000 -1.95 -1.10300003 rpy=0 0 0 -> xyz=0.000000 -1.95 -1.25 rpy=0 0 0

Commit message: Update parameters 3dofs

File: resources/urdf/pps.urdf (robot description, URDF)
Before this commit: robot test_robot, 5 links, 4 joints
Joints:
- joint base: origin xyz=0.000000 -1.95 -1.10300003 rpy=0 0 0 -> xyz=0.000000 -1.95 -1.25 rpy=0 0 0
- joint joint1: origin xyz=-1.2 0 0.36 rpy=0 0 0 -> xyz=-1.2 0 0.4365 rpy=0 0 0
- joint joint2: origin xyz=0.36 0 0.27 rpy=0 0 0 -> xyz=0.36 0 0.1935 rpy=0 0 0
